File: Project/_autosave-巻き線切り替え回路.kicad_pcb (KiCad board)
At the start: 2 copper layers, 237.5 x 168.9 mm, 155 parts, among them U2 IRLU024N

Commit message: フォルダ整理
Parts:
- added Relay: 0-1432871-1, Kageyama_Device:0-1432871-1, F.Cu at (296.6, 62.6)
