File: Project/巻き線切り替え回路.kicad_pcb (KiCad board)
At the start: 2 copper layers, 237.5 x 168.9 mm, 155 parts, among them U2 IRLU024N

Commit message: 長穴連打実装
Parts:
- moved hole 0.25 mm to (222.5, 37.5)
Routing:
- net /RCSout: track 714.8 -> 731.1 mm
